File: hw/leddimmer-hw.kicad_pcb (KiCad board)
At the start: 4 copper layers, 52 x 80 mm, 117 parts, among them J401 2604-1102, J402 2604-1102, J403 2604-1102, J404 2604-1102, P401 TYPE-C-31-M-12, Q201 CSD17571Q2, Q301 CSD17571Q2, U201 NCV8460A, U202 UCC27511DBVR, U203 INA2180A2IDGKR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

Commit message: Fixed some bugs
Parts:
- moved H102 7.00 mm to (109.0, 59.5)
- moved C605 4.30 mm to (107.5, 107.0), turned to -90 degrees
- moved R604 4.30 mm to (105.5, 107.0), turned to -90 degrees
- moved R605 4.30 mm to (106.5, 107.0), turned to 90 degrees
Routing:
- net /MCU/24V_MEAS: track 53.0 -> 48.3 mm
- net +24V: track 14.0 -> 18.1 mm
Other:
- board text added: "24V IN"
- board text added: "24V OUT"
- board text added: "DRV1"
- board text added: "DRV2"
